File: kicad/kicad.kicad_pcb (KiCad board)
At the start: 0 parts

Commit message: Session #1: README update, designed the whole board lol
Parts:
- added BT2: Battery_Cell, Battery:BatteryHolder_MYOUNG_BS-07-A1BJ001_CR2032, B.Cu at (141.0, 99.5)
- added D1: LED, LED_THT:LED_D5.0mm, F.Cu at (122.5, 70.5)
- added D10: LED, LED_THT:LED_D5.0mm, F.Cu at (111.5, 83.0)
- added D2: LED, LED_THT:LED_D5.0mm, F.Cu at (141.0, 84.0)
- added D3: LED, LED_THT:LED_D5.0mm, F.Cu at (159.0, 70.5)
- added D4: LED, LED_THT:LED_D5.0mm, F.Cu at (170.0, 83.0)
- added D5: LED, LED_THT:LED_D5.0mm, F.Cu at (165.0, 101.0)
- added D6: LED, LED_THT:LED_D5.0mm, F.Cu at (155.5, 113.5)
- added D7: LED, LED_THT:LED_D5.0mm, F.Cu at (141.0, 127.5)
- added D8: LED, LED_THT:LED_D5.0mm, F.Cu at (126.5, 113.5)
- added D9: LED, LED_THT:LED_D5.0mm, F.Cu at (117.0, 101.0)
- added R1: 220, Resistor_THT:R_Axial_DIN0207_L6.3mm_D2.5mm_P10.16mm_Horizontal, B.Cu at (155.0, 92.0)
- added R2: 10k, Resistor_THT:R_Axial_DIN0207_L6.3mm_D2.5mm_P10.16mm_Horizontal, B.Cu at (131.5, 100.5)
- added RV1: Trimpot, Potentiometer_THT:Potentiometer_Runtron_RM-065_Vertical, B.Cu at (129.0, 82.5)
- added SW1: SW_Push, Button_Switch_THT:SW_PUSH_6mm, F.Cu at (137.5, 89.0)
- added U2: ATtiny85-20P, Package_DIP:DIP-8_W7.62mm, B.Cu at (162.5, 78.5)
Routing:
- net Net-(D1-A): track 0.00 -> 194.8 mm, vias 0 -> 1
- net GND: track 0.00 -> 193.0 mm, vias 0 -> 3
- net Net-(U2-XTAL1/PB3): track 0.00 -> 44.0 mm
- net Net-(BT2-+): track 0.00 -> 36.7 mm
- net Net-(U2-PB1): track 0.00 -> 9.38 mm
- net Net-(U2-PB2): track 0.00 -> 6.50 mm
- added copper zone on B.Cu, net GND
Other:
- board outline added: 70 x 70 mm
- copper layers 0 -> 2
- board text added: "(I love you xx)"
- board text added: "For: Jam Jam"
- board text added: "From: Pence"
